File: pcb/toroufc.kicad_sch (KiCad schematic)
At the start: 64 parts, among them J1 Conn_01x16_Male, J3 Conn_01x16_Male, J4 Conn_01x16_Male, J5 Conn_01x16_Male, J6 Conn_01x16_Male, J7 Conn_01x16_Male, J8 Conn_01x16_Male, J9 Conn_01x16_Male

Commit message: Moving stuff.
Parts:
- removed J1: Conn_01x16_Male, Connector_PinHeader_2.54mm:PinHeader_1x16_P2.54mm_Vertical, symbol Connector:Conn_01x16_Male
- added J8, J9: Conn_01x09_Male, symbol Connector:Conn_01x09_Male
- added J?: USB_B_Mini, symbol Connector:USB_B_Mini
- added U1: YAAJ_BluePill, bluepill:YAAJ_BluePill_1, symbol bluepill:YAAJ_BluePill
- renumbered J3 to J1, J4 to J2, J5 to J3, J6 to J4, J7 to J5, J8 to J6, J9 to J7
Connections:
- net COL7: now reaches J7.10 (Pin_10), J7.12 (Pin_12), J7.14 (Pin_14), J7.16 (Pin_16), J7.2 (Pin_2), J7.4 (Pin_4), J7.6 (Pin_6), J7.8 (Pin_8)
- net COL7: now also U1.5 (PA8)
- net COL6: now reaches J6.10 (Pin_10), J6.12 (Pin_12), J6.14 (Pin_14), J6.16 (Pin_16), J6.2 (Pin_2), J6.4 (Pin_4), J6.6 (Pin_6), J6.8 (Pin_8)
- net COL6: now also U1.6 (PA9)
- net COL5: now reaches J5.10 (Pin_10), J5.12 (Pin_12), J5.14 (Pin_14), J5.16 (Pin_16), J5.2 (Pin_2), J5.4 (Pin_4), J5.6 (Pin_6), J5.8 (Pin_8)
- net COL5: now also U1.7 (PA10)
- net COL4: now reaches J4.10 (Pin_10), J4.12 (Pin_12), J4.14 (Pin_14), J4.16 (Pin_16), J4.2 (Pin_2), J4.4 (Pin_4), J4.6 (Pin_6), J4.8 (Pin_8)
- net COL4: now also U1.10 (PA15)
- net COL3: now reaches J3.10 (Pin_10), J3.12 (Pin_12), J3.14 (Pin_14), J3.16 (Pin_16), J3.2 (Pin_2), J3.4 (Pin_4), J3.6 (Pin_6), J3.8 (Pin_8)
- net COL3: now also U1.11 (PB3)
- net COL2: now reaches J2.10 (Pin_10), J2.12 (Pin_12), J2.14 (Pin_14), J2.16 (Pin_16), J2.2 (Pin_2), J2.4 (Pin_4), J2.6 (Pin_6), J2.8 (Pin_8)
- net COL2: now also U1.12 (PB4)
- net COL1: now reaches J1.10 (Pin_10), J1.12 (Pin_12), J1.14 (Pin_14), J1.16 (Pin_16), J1.2 (Pin_2), J1.4 (Pin_4), J1.6 (Pin_6), J1.8 (Pin_8)
- net COL1: now also U1.13 (PB5)
- net ROW8: now reaches D1.1 (K), D17.1 (K), D25.1 (K), D33.1 (K), D41.1 (K), D49.1 (K), D9.1 (K)
- net ROW8: now also U1.16 (PB8)
- net ROW7: now reaches D10.1 (K), D18.1 (K), D2.1 (K), D26.1 (K), D34.1 (K), D42.1 (K), D50.1 (K)
- net ROW7: now also U1.17 (PB9)
- net ROW6: now reaches D11.1 (K), D19.1 (K), D27.1 (K), D3.1 (K), D35.1 (K), D43.1 (K), D51.1 (K)
- net ROW6: now also U1.36 (PB11)
- net ROW5: now reaches D12.1 (K), D20.1 (K), D28.1 (K), D36.1 (K), D4.1 (K), D44.1 (K), D52.1 (K)
- net ROW5: now also U1.35 (PB10)
- net ROW4: now reaches D13.1 (K), D21.1 (K), D29.1 (K), D37.1 (K), D45.1 (K), D5.1 (K), D53.1 (K)
- net ROW4: now also U1.34 (PB1)
- net ROW3: now reaches D14.1 (K), D22.1 (K), D30.1 (K), D38.1 (K), D46.1 (K), D54.1 (K), D6.1 (K)
- net ROW3: now also U1.33 (PB0)
- net ROW2: now reaches D15.1 (K), D23.1 (K), D31.1 (K), D39.1 (K), D47.1 (K), D55.1 (K), D7.1 (K)
- net ROW2: now also U1.32 (PA7)
- net ROW1: now reaches D16.1 (K), D24.1 (K), D32.1 (K), D40.1 (K), D48.1 (K), D56.1 (K), D8.1 (K)
- net ROW1: now also U1.31 (PA6)
- new net GND: J8.1 (Pin_1), J8.4 (Pin_4), J8.7 (Pin_7), J9.1 (Pin_1), J9.4 (Pin_4), J9.7 (Pin_7), J?.5 (GND), U1.19 (GND), U1.39 (GND), U1.40 (GND)
- new net POT1: J8.8 (Pin_8), U1.30 (PA5)
- new net POT2: J8.5 (Pin_5), U1.29 (PA4)
- new net POT3: J8.2 (Pin_2), U1.28 (PA3)
- new net POT4: J9.8 (Pin_8), U1.27 (PA2)
- new net POT5: J9.5 (Pin_5), U1.26 (PA1)
- new net POT6: J9.2 (Pin_2), U1.25 (PA0)
- new net ROT1C: U1.2 (PB13)
- new net ROT1D: U1.1 (PB12)
- new net ROT2C: U1.4 (PB15)
- new net ROT2D: U1.3 (PB14)
- new net SCL: U1.14 (PB6)
- new net SDA: U1.15 (PB7)
- new net USBD+: J?.3 (D+), U1.9 (PA12)
- new net USBD-: J?.2 (D-), U1.8 (PA11)
- new net VCC: J8.3 (Pin_3), J8.6 (Pin_6), J8.9 (Pin_9), J9.3 (Pin_3), J9.6 (Pin_6), J9.9 (Pin_9), J?.1 (VBUS), U1.18 (5V)

Commit message: More rinsing.
Parts:
- gave numbers to parts that had none: 1
Connections:
- net ROT1C renamed REN1C
- net ROT1D renamed REN1D
- net ROT2C renamed REN2C
- net ROT2D renamed REN2D
Other:
- note added: "COLUMNS are set as inputs with pullup ROWS are set as HIGH outputs, except for the one scanning, which will be set as LOW output. The corresponding column with a switch pressed will be set to low, the unpressed ones will remain high."
- note added: "REN lines go to rotary encoders POT lines go to potentiometers ROW lines are the rows of the scan matrix COL lines are the columns of the scan matrix"
