File: pcb/main/toroufc.kicad_sch (KiCad schematic)
At the start: 39 parts, among them J1 HAT, J10 RPAD, J11 POT1-3, J12 POT4-6, J13 REN1, J14 REN2, J15 I2C, J16 Conn_01x04_Male, J2 RKR1-2, J3 RKR3-4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

Commit message: Added test points, reduced size, removed i2c, labels, bluepill fix.
Parts:
- removed J15: I2C, Connector_JST:JST_XH_B4B-XH-A_1x04_P2.50mm_Vertical, symbol Connector:Conn_01x04_Male
- added R1: R1.5K, Resistor_SMD:R_0805_2012Metric_Pad1.20x1.40mm_HandSolder, symbol Device:R
- added TP1: VCC, TestPoint:TestPoint_Pad_2.0x2.0mm, symbol Connector:TestPoint
- added TP2: Vusb, TestPoint:TestPoint_Pad_2.0x2.0mm, symbol Connector:TestPoint
- added TP3: GND, TestPoint:TestPoint_Pad_2.0x2.0mm, symbol Connector:TestPoint
- J16: value Conn_01x04_Male -> USB connector
Connections:
- net GND: now also TP3.1
- net ROW7: now also U1.16 (PB8); no longer U1.17 (PB9)
- net ROW8: now also U1.17 (PB9); no longer U1.16 (PB8)
- net USBD+: now also R1.1
- net VCC: now also R1.2, TP1.1
- net Vusb: now also TP2.1
Other:
- note added: "Bluepill USB fix (see https://stm32duinoforum.com/forum/wiki_subdomain/index_title_Blue_Pill.html#Known_issues)"
