File: pcb/hpad/toroufc-hpad.kicad_pcb (KiCad board)
At the start: 2 copper layers, 163.5 x 21.5 mm, 15 parts, among them J1 Conn_01x08_Male, SW1 SW_Push, SW2 SW_Push, SW3 SW_Push, SW4 SW_Push, SW5 SW_Push, SW6 SW_Push, SW7 SW_Push

Commit message: Preparing PCBs v2
Connections:
- J1 pad 1: /COL1 -> /ROW7
- J1 pad 2: /ROW1 -> /ROW6
- J1 pad 3: /ROW2 -> /ROW5
- J1 pad 4: /ROW3 -> /ROW4
- J1 pad 5: /ROW4 -> /ROW3
- J1 pad 6: /ROW5 -> /ROW2
- J1 pad 7: /ROW6 -> /ROW1
- J1 pad 8: /ROW7 -> /COL1
Routing:
- net /ROW7: track 76.8 -> 193.0 mm
- net /ROW6: track 47.2 -> 159.7 mm
- net /ROW1: track 45.8 -> 62.9 mm
- net /ROW5: track 29.2 -> 45.6 mm
- net /ROW2: track 28.3 -> 43.2 mm
- net /ROW4: track 5.08 -> 10.1 mm
- net /ROW3: track 4.81 -> 5.85 mm
- net /COL1: track 159.3 -> 158.3 mm
Other:
- board text added: "UFC-HPAD v2 2022"
- board text removed: "UFC-HPAD v1 2022"
