File: pcb/hpad/toroufc-hpad.kicad_sch (KiCad schematic)
At the start: 15 parts, among them J1 Conn_01x08_Male, SW1 SW_Push, SW2 SW_Push, SW3 SW_Push, SW4 SW_Push, SW5 SW_Push, SW6 SW_Push, SW7 SW_Push

Commit message: Preparing PCBs v2
Connections:
- net COL1: now also J1.8 (Pin_8); no longer J1.1 (Pin_1)
- net ROW1: now also J1.7 (Pin_7); no longer J1.2 (Pin_2)
- net ROW2: now also J1.6 (Pin_6); no longer J1.3 (Pin_3)
- net ROW3: now also J1.5 (Pin_5); no longer J1.4 (Pin_4)
- net ROW4: now also J1.4 (Pin_4); no longer J1.5 (Pin_5)
- net ROW5: now also J1.3 (Pin_3); no longer J1.6 (Pin_6)
- net ROW6: now also J1.2 (Pin_2); no longer J1.7 (Pin_7)
- net ROW7: now also J1.1 (Pin_1); no longer J1.8 (Pin_8)
Changed lines of the file:
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@@
     (stroke (width 0) (type default) (color 0 0 0 0))
   )
-  (label "COL1" (at 108.5923 72.644 0)
+  (label "COL1" (at 108.5138 90.424 0)
     (effects (font (size 1.27 1.27)) (justify left bottom))
   )
@@
     (effects (font (size 1.27 1.27)) (justify left bottom))
   )
-  (label "ROW3" (at 108.5357 80.264 0)
+  (label "ROW3" (at 108.5138 82.804 0)
     (effects (font (size 1.27 1.27)) (justify left bottom))
   )
@@
     (effects (font (size 1.27 1.27)) (justify left bottom))
   )
-  (label "ROW4" (at 108.5138 82.804 0)
+  (label "ROW4" (at 108.5357 80.264 0)
     (effects (font (size 1.27 1.27)) (justify left bottom))
   )
-  (label "ROW1" (at 108.5923 75.184 0)
+  (label "ROW1" (at 108.5138 87.884 0)
     (effects (font (size 1.27 1.27)) (justify left bottom))
   )
@@
     (effects (font (size 1.27 1.27)) (justify left bottom))
   )
-  (label "ROW7" (at 108.5138 90.424 0)
+  (label "ROW7" (at 108.5923 72.644 0)
     (effects (font (size 1.27 1.27)) (justify left bottom))
   )
@@
     (effects (font (size 1.27 1.27)) (justify left bottom))
   )
-  (label "ROW6" (at 108.5138 87.884 0)
+  (label "ROW6" (at 108.5923 75.184 0)
     (effects (font (size 1.27 1.27)) (justify left bottom))
   )
-  (label "ROW5" (at 108.5138 85.3452 0)
+  (label "ROW5" (at 108.5357 77.7232 0)
     (effects (font (size 1.27 1.27)) (justify left bottom))
   )
@@
     (effects (font (size 1.27 1.27)) (justify left bottom))
   )
-  (label "ROW2" (at 108.5357 77.7232 0)
+  (label "ROW2" (at 108.5138 85.3452 0)
     (effects (font (size 1.27 1.27)) (justify left bottom))
   )
