File: pcb/lpad/toroufc-lpad.kicad_pcb (KiCad board)
At the start: 2 copper layers, 20 x 109.2 mm, 11 parts, among them J1 Conn_01x06_Male, SW1 SW_Push, SW2 SW_Push, SW3 SW_Push, SW4 SW_Push, SW5 SW_Push

Commit message: First production
Routing:
- added copper zone on B.Cu, net (none)
- added copper zone on F.Cu, net (none)
- removed copper zone on F.Cu, net /COL4
Other:
- board text added: "UFC-LPAD v1 2022"
- board text removed: "Toro UFC LPAD"
Changed lines of the file:
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@@
     (pad_to_mask_clearance 0)
     (pcbplotparams
-      (layerselection 0x00010fc_ffffffff)
+      (layerselection 0x00010f0_ffffffff)
       (disableapertmacros false)
       (usegerberextensions false)
@@
       (outputformat 1)
       (mirror false)
-      (drillshape 1)
+      (drillshape 0)
       (scaleselection 1)
-      (outputdirectory "")
+      (outputdirectory "production/")
     )
   )
@@
     (fp_line (start 0 1.35) (end 0.625 2.35) (layer "B.Fab") (width 0.1))
     (fp_line (start -0.625 2.35) (end 0 1.35) (layer "B.Fab") (width 0.1))
-    (pad "1" thru_hole roundrect (at 0 0) (size 1.7 1.95) (drill 0.95) (layers *.Cu *.Mask) (roundrect_rratio 0.147059)
+    (pad "1" thru_hole roundrect (at 0 0) (size 1.7 1.95) (drill 0.95) (layers *.Cu *.Mask) (roundrect_rratio 0.1470588235)
       (net 10 "/COL4") (pinfunction "Pin_1") (pintype "passive"))
     (pad "2" thru_hole oval (at 2.5 0) (size 1.7 1.95) (drill 0.95) (layers *.Cu *.Mask)
@@
   )
   (gr_rect (start 140 30) (end 160 139.25) (layer "Edge.Cuts") (width 0.1) (fill none))
-  (gr_text "Toro UFC LPAD" (at 150 32) (layer "B.SilkS")
-    (effects (font (size 1.5 1.5) (thickness 0.3)) (justify mirror))
+  (gr_text "UFC-LPAD v1\n2022" (at 142.5 33.3) (layer "B.SilkS")
+    (effects (font (size 1.5 1.5) (thickness 0.3)) (justify right mirror))
+  )
+  (dimension (type aligned) (layer "Cmts.User")
+    (pts (xy 140 139.25) (xy 160 139.25))
+    (height 5.1744)
+    (gr_text "20.0000 mm" (at 150 143.2744) (layer "Cmts.User")
+      (effects (font (size 1 1) (thickness 0.15)))
+    )
+    (format (units 3) (units_format 1) (precision 4))
+    (style (thickness 0.15) (arrow_length 1.27) (text_position_mode 0) (extension_height 0.58642) (extension_offset 0.5) keep_text_aligned)
+  )
+  (dimension (type aligned) (layer "Cmts.User")
+    (pts (xy 160 30) (xy 160 139.25))
+    (height -4.7952)
+    (gr_text "109.2500 mm" (at 163.6452 84.625 90) (layer "Cmts.User")
+      (effects (font (size 1 1) (thickness 0.15)))
+    )
+    (format (units 3) (units_format 1) (precision 4))
+    (style (thickness 0.15) (arrow_length 1.27) (text_position_mode 0) (extension_height 0.58642) (extension_offset 0.5) keep_text_aligned)
   )
   (segment (start 152.54 45.31) (end 152.5 45.35) (width 0.25) (layer "B.Cu") (net 1))
@@
   (segment (start 152.5 125.35) (end 152.5 114.96) (width 0.25) (layer "B.Cu") (net 11))
   (segment (start 152.5 114.96) (end 152.54 114.92) (width 0.25) (layer "B.Cu") (net 11))
-  (zone (net 10) (net_name "/COL4") (layer "F.Cu") (hatch edge 0.508)
+  (zone (net 0) (net_name "") (layers F&B.Cu) (hatch edge 0.508)
     (connect_pads (clearance 0.508))
     (min_thickness 0.254) (filled_areas_thickness no)

Commit message: Preparing PCBs v2
Connections:
- J1 pad 1: /COL4 -> /ROW5
- J1 pad 2: /ROW1 -> /ROW4
- J1 pad 3: /ROW2 -> /ROW3
- J1 pad 4: /ROW3 -> /ROW2
- J1 pad 5: /ROW4 -> /ROW1
- J1 pad 6: /ROW5 -> /COL4
Routing:
- net /COL4: track 115.2 -> 228.6 mm
- net /ROW1: track 98.7 -> 93.1 mm
- net /ROW2: track 78.5 -> 74.2 mm
- net /ROW5: track 9.27 -> 13.2 mm
- net /ROW3: track 58.5 -> 55.9 mm
- net /ROW4: track 38.8 -> 36.3 mm
Other:
- board text added: "UFC-LPAD v2 2022"
- board text removed: "UFC-LPAD v1 2022"
