File: pcb/lpad/toroufc-lpad.kicad_sch (KiCad schematic)
At the start: 11 parts, among them J1 Conn_01x06_Male, SW1 SW_Push, SW2 SW_Push, SW3 SW_Push, SW4 SW_Push, SW5 SW_Push

Commit message: Preparing PCBs v2
Connections:
- net COL4: now also J1.6 (Pin_6); no longer J1.1 (Pin_1)
- net ROW1: now also J1.5 (Pin_5); no longer J1.2 (Pin_2)
- net ROW2: now also J1.4 (Pin_4); no longer J1.3 (Pin_3)
- net ROW3: now also J1.3 (Pin_3); no longer J1.4 (Pin_4)
- net ROW4: now also J1.2 (Pin_2); no longer J1.5 (Pin_5)
- net ROW5: now also J1.1 (Pin_1); no longer J1.6 (Pin_6)
Changed lines of the file:
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@@
     (stroke (width 0) (type default) (color 0 0 0 0))
   )
-  (label "COL4" (at 113.8448 88.773 0)
+  (label "COL4" (at 113.7663 101.4742 0)
     (effects (font (size 1.27 1.27)) (justify left bottom))
   )
@@
     (effects (font (size 1.27 1.27)) (justify left bottom))
   )
-  (label "ROW3" (at 113.7882 96.393 0)
+  (label "ROW3" (at 113.7882 93.8522 0)
     (effects (font (size 1.27 1.27)) (justify left bottom))
   )
-  (label "ROW4" (at 113.7663 98.933 0)
+  (label "ROW4" (at 113.8448 91.313 0)
     (effects (font (size 1.27 1.27)) (justify left bottom))
   )
-  (label "ROW1" (at 113.8448 91.313 0)
+  (label "ROW1" (at 113.7663 98.933 0)
     (effects (font (size 1.27 1.27)) (justify left bottom))
   )
@@
     (effects (font (size 1.27 1.27)) (justify left bottom))
   )
-  (label "ROW5" (at 113.7663 101.4742 0)
+  (label "ROW5" (at 113.8448 88.773 0)
     (effects (font (size 1.27 1.27)) (justify left bottom))
   )
@@
     (effects (font (size 1.27 1.27)) (justify left bottom))
   )
-  (label "ROW2" (at 113.7882 93.8522 0)
+  (label "ROW2" (at 113.7882 96.393 0)
     (effects (font (size 1.27 1.27)) (justify left bottom))
   )
