File: pcb/npad/toroufc-npad.kicad_pcb (KiCad board)
At the start: 2 copper layers, 55.9 x 80.9 mm, 25 parts, among them J1 Conn_01x10_Male, SW0 SW_Push, SW1 SW_Push, SW2 SW_Push, SW3 SW_Push, SW4 SW_Push, SW5 SW_Push, SW6 SW_Push, SW7 SW_Push, SW8 SW_Push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

Commit message: Preparing PCBs v2
Parts:
- moved J1 22.5 mm to (131.3, 128.8), turned to 180 degrees
Connections:
- J1 pad 1: /COL2 -> /ROW8
- J1 pad 10: /ROW8 -> /COL2
- J1 pad 2: /COL3 -> /ROW7
- J1 pad 3: /ROW1 -> /ROW6
- J1 pad 4: /ROW2 -> /ROW5
- J1 pad 5: /ROW3 -> /ROW4
- J1 pad 6: /ROW4 -> /ROW3
- J1 pad 7: /ROW5 -> /ROW2
- J1 pad 8: /ROW6 -> /ROW1
- J1 pad 9: /ROW7 -> /COL3
Routing:
- net /ROW4: track 81.4 -> 82.8 mm
- net /ROW7: track 44.5 -> 43.3 mm
Other:
- board text added: "UFC-NPAD v2 2022"
- board text removed: "UFC-NPAD v1 2022"
Changed lines of the file:
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@@
   )
   (footprint "Connector_JST:JST_XH_B10B-XH-AM_1x10_P2.50mm_Vertical" (layer "B.Cu")
-    (at 108.7882 128.8542)
+    (at 131.3 128.8 180)
     (descr "JST XH series connector, B10B-XH-AM, with boss (http://www.jst-mfg.com/product/pdf/eng/eXH.pdf), generated with kicad-footprint-generator")
     (tags "connector JST XH side entry boss")
@@
     (property "Sheetname" "")
     (attr through_hole)
-    (fp_text reference "J1" (at -0.381 -4.445) (layer "B.SilkS")
+    (fp_text reference "J1" (at 10.2 3.2) (layer "B.SilkS")
       (effects (font (size 1 1) (thickness 0.15)) (justify mirror))
     )
@@
     (fp_line (start -0.625 2.35) (end 0 1.35) (layer "B.Fab") (width 0.1))
     (fp_line (start 24.95 -3.4) (end 24.95 2.35) (layer "B.Fab") (width 0.1))
-    (pad "" np_thru_hole circle (at -1.6 -2) (size 1.2 1.2) (drill 1.2) (layers *.Cu *.Mask))
-    (pad "1" thru_hole roundrect (at 0 0) (size 1.7 1.95) (drill 0.95) (layers *.Cu *.Mask) (roundrect_rratio 0.1470588235)
-      (net 20 "/COL2") (pinfunction "Pin_1") (pintype "passive"))
-    (pad "2" thru_hole oval (at 2.5 0) (size 1.7 1.95) (drill 0.95) (layers *.Cu *.Mask)
-      (net 21 "/COL3") (pinfunction "Pin_2") (pintype "passive"))
-    (pad "3" thru_hole oval (at 5 0) (size 1.7 1.95) (drill 0.95) (layers *.Cu *.Mask)
-      (net 3 "/ROW1") (pinfunction "Pin_3") (pintype "passive"))
-    (pad "4" thru_hole oval (at 7.5 0) (size 1.7 1.95) (drill 0.95) (layers *.Cu *.Mask)
-      (net 1 "/ROW2") (pinfunction "Pin_4") (pintype "passive"))
-    (pad "5" thru_hole oval (at 10 0) (size 1.7 1.95) (drill 0.95) (layers *.Cu *.Mask)
-      (net 6 "/ROW3") (pinfunction "Pin_5") (pintype "passive"))
-    (pad "6" thru_hole oval (at 12.5 0) (size 1.7 1.95) (drill 0.95) (layers *.Cu *.Mask)
-      (net 7 "/ROW4") (pinfunction "Pin_6") (pintype "passive"))
-    (pad "7" thru_hole oval (at 15 0) (size 1.7 1.95) (drill 0.95) (layers *.Cu *.Mask)
-      (net 9 "/ROW5") (pinfunction "Pin_7") (pintype "passive"))
-    (pad "8" thru_hole oval (at 17.5 0) (size 1.7 1.95) (drill 0.95) (layers *.Cu *.Mask)
-      (net 11 "/ROW6") (pinfunction "Pin_8") (pintype "passive"))
-    (pad "9" thru_hole oval (at 20 0) (size 1.7 1.95) (drill 0.95) (layers *.Cu *.Mask)
-      (net 13 "/ROW7") (pinfunction "Pin_9") (pintype "passive"))
-    (pad "10" thru_hole oval (at 22.5 0) (size 1.7 1.95) (drill 0.95) (layers *.Cu *.Mask)
-      (net 15 "/ROW8") (pinfunction "Pin_10") (pintype "passive"))
+    (pad "" np_thru_hole circle (at -1.6 -2 180) (size 1.2 1.2) (drill 1.2) (layers *.Cu *.Mask))
+    (pad "1" thru_hole roundrect (at 0 0 180) (size 1.7 1.95) (drill 0.95) (layers *.Cu *.Mask) (roundrect_rratio 0.1470588235)
+      (net 15 "/ROW8") (pinfunction "Pin_1") (pintype "passive"))
+    (pad "2" thru_hole oval (at 2.5 0 180) (size 1.7 1.95) (drill 0.95) (layers *.Cu *.Mask)
+      (net 13 "/ROW7") (pinfunction "Pin_2") (pintype "passive"))
+    (pad "3" thru_hole oval (at 5 0 180) (size 1.7 1.95) (drill 0.95) (layers *.Cu *.Mask)
+      (net 11 "/ROW6") (pinfunction "Pin_3") (pintype "passive"))
+    (pad "4" thru_hole oval (at 7.5 0 180) (size 1.7 1.95) (drill 0.95) (layers *.Cu *.Mask)
+      (net 9 "/ROW5") (pinfunction "Pin_4") (pintype "passive"))
+    (pad "5" thru_hole oval (at 10 0 180) (size 1.7 1.95) (drill 0.95) (layers *.Cu *.Mask)
+      (net 7 "/ROW4") (pinfunction "Pin_5") (pintype "passive"))
+    (pad "6" thru_hole oval (at 12.5 0 180) (size 1.7 1.95) (drill 0.95) (layers *.Cu *.Mask)
+      (net 6 "/ROW3") (pinfunction "Pin_6") (pintype "passive"))
+    (pad "7" thru_hole oval (at 15 0 180) (size 1.7 1.95) (drill 0.95) (layers *.Cu *.Mask)
+      (net 1 "/ROW2") (pinfunction "Pin_7") (pintype "passive"))
+    (pad "8" thru_hole oval (at 17.5 0 180) (size 1.7 1.95) (drill 0.95) (layers *.Cu *.Mask)
+      (net 3 "/ROW1") (pinfunction "Pin_8") (pintype "passive"))
+    (pad "9" thru_hole oval (at 20 0 180) (size 1.7 1.95) (drill 0.95) (layers *.Cu *.Mask)
+      (net 21 "/COL3") (pinfunction "Pin_9") (pintype "passive"))
+    (pad "10" thru_hole oval (at 22.5 0 180) (size 1.7 1.95) (drill 0.95) (layers *.Cu *.Mask)
+      (net 20 "/COL2") (pinfunction "Pin_10") (pintype "passive"))
     (model "${KICAD6_3DMODEL_DIR}/Connector_JST.3dshapes/JST_XH_B10B-XH-A_1x10_P2.50mm_Vertical.wrl"
       (offset (xyz 0 0 0))
@@
   )
   (gr_rect (start 92.0496 51.8414) (end 147.9042 132.7912) (layer "Edge.Cuts") (width 0.1) (fill none))
-  (gr_text "UFC-NPAD v1\n2022" (at 133.6 71.3) (layer "B.SilkS")
+  (gr_text "UFC-NPAD v2\n2022" (at 133.6 71.3) (layer "B.SilkS")
     (effects (font (size 1.5 1.5) (thickness 0.3)) (justify mirror))
   )
@@
   (segment (start 121.2374 128.905) (end 121.2374 128.5526) (width 0.25) (layer "F.Cu") (net 7))
   (via (at 113.7666 121.9454) (size 0.8) (drill 0.4) (layers "F.Cu" "B.Cu") (net 7))
+  (segment (start 131.321818 131) (end 132.496339 129.825479) (width 0.25) (layer "B.Cu") (net 7))
   (segment (start 101.5238 104.8766) (end 105.8926 104.8766) (width 0.25) (layer "B.Cu") (net 7))
   (segment (start 100.5332 108.712) (end 100.5332 105.8672) (width 0.25) (layer "B.Cu") (net 7))
-  (segment (start 123.4208 131.0884) (end 121.2374 128.905) (width 0.25) (layer "B.Cu") (net 7))
+  (segment (start 121.3 129.5) (end 122.8 131) (width 0.25) (layer "B.Cu") (net 7))
   (segment (start 105.8926 104.8766) (end 107.2642 103.505) (width 0.25) (layer "B.Cu") (net 7))
-  (segment (start 123.4208 131.0884) (end 143.2052 131.0884) (width 0.25) (layer "B.Cu") (net 7))
+  (segment (start 139.3884 131.0884) (end 143.2052 131.0884) (width 0.25) (layer "B.Cu") (net 7))
+  (segment (start 122.8 131) (end 131.321818 131) (width 0.25) (layer "B.Cu") (net 7))
+  (segment (start 121.3 128.8) (end 121.3 129.5) (width 0.25) (layer "B.Cu") (net 7))
   (segment (start 113.7666 121.9454) (end 100.5332 108.712) (width 0.25) (layer "B.Cu") (net 7))
+  (segment (start 132.496339 129.825479) (end 138.125479 129.825479) (width 0.25) (layer "B.Cu") (net 7))
   (segment (start 100.5332 105.8672) (end 101.5238 104.8766) (width 0.25) (layer "B.Cu") (net 7))
   (segment (start 107.2642 103.505) (end 107.2642 90.7278) (width 0.25) (layer "B.Cu") (net 7))
+  (segment (start 138.125479 129.825479) (end 139.3884 131.0884) (width 0.25) (layer "B.Cu") (net 7))
   (segment (start 107.2642 90.7278) (end 103.0732 86.5368) (width 0.25) (layer "B.Cu") (net 7))
   (segment (start 103.0732 75.4532) (end 102.54 74.92) (width 0.25) (layer "B.Cu") (net 8))
@@
   (segment (start 143.2052 75.5852) (end 142.54 74.92) (width 0.25) (layer "B.Cu") (net 12))
   (segment (start 143.2052 83.186) (end 143.2052 75.5852) (width 0.25) (layer "B.Cu") (net 12))
-  (segment (start 122.56288 130.48768) (end 123.1646 131.0894) (width 0.25) (layer "F.Cu") (net 13))
-  (segment (start 126.553 131.0894) (end 128.7374 128.905) (width 0.25) (layer "F.Cu") (net 13))
-  (segment (start 123.1646 131.0894) (end 126.553 131.0894) (width 0.25) (layer "F.Cu") (net 13))
+  (segment (start 122.56288 122.47092) (end 122.56288 129.56288) (width 0.25) (layer "F.Cu") (net 13))
+  (segment (start 122.56288 129.56288) (end 123.3 130.3) (width 0.25) (layer "F.Cu") (net 13))
+  (segment (start 127.3424 130.3) (end 128.7374 128.905) (width 0.25) (layer "F.Cu") (net 13))
   (segment (start 123.1138 121.92) (end 122.56288 122.47092) (width 0.25) (layer "F.Cu") (net 13))
-  (segment (start 122.56288 122.47092) (end 122.56288 130.48768) (width 0.25) (layer "F.Cu") (net 13))
+  (segment (start 123.3 130.3) (end 127.3424 130.3) (width 0.25) (layer "F.Cu") (net 13))
   (via (at 123.1138 121.92) (size 0.8) (drill 0.4) (layers "F.Cu" "B.Cu") (net 13))
   (segment (start 123.1138 118.4656) (end 111.2002 106.552) (width 0.25) (layer "B.Cu") (net 13))
