File: pcb/npad/toroufc-npad.kicad_sch (KiCad schematic)
At the start: 25 parts, among them J1 Conn_01x10_Male, SW0 SW_Push, SW1 SW_Push, SW2 SW_Push, SW3 SW_Push, SW4 SW_Push, SW5 SW_Push, SW6 SW_Push, SW7 SW_Push, SW8 SW_Push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

Commit message: Preparing PCBs v2
Connections:
- net COL2: now also J1.10 (Pin_10); no longer J1.1 (Pin_1)
- net COL3: now also J1.9 (Pin_9); no longer J1.2 (Pin_2)
- net ROW1: now also J1.8 (Pin_8); no longer J1.3 (Pin_3)
- net ROW2: now also J1.7 (Pin_7); no longer J1.4 (Pin_4)
- net ROW3: now also J1.6 (Pin_6); no longer J1.5 (Pin_5)
- net ROW4: now also J1.5 (Pin_5); no longer J1.6 (Pin_6)
- net ROW5: now also J1.4 (Pin_4); no longer J1.7 (Pin_7)
- net ROW6: now also J1.3 (Pin_3); no longer J1.8 (Pin_8)
- net ROW7: now also J1.2 (Pin_2); no longer J1.9 (Pin_9)
- net ROW8: now also J1.1 (Pin_1); no longer J1.10 (Pin_10)
Changed lines of the file:
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@@
     (stroke (width 0) (type default) (color 0 0 0 0))
   )
-  (label "COL2" (at 113.8448 88.773 0)
+  (label "COL2" (at 113.7663 111.633 0)
     (effects (font (size 1.27 1.27)) (justify left bottom))
   )
@@
     (effects (font (size 1.27 1.27)) (justify left bottom))
   )
-  (label "ROW8" (at 113.7663 111.633 0)
+  (label "ROW8" (at 113.8448 88.773 0)
     (effects (font (size 1.27 1.27)) (justify left bottom))
   )
-  (label "ROW2" (at 113.7882 96.393 0)
+  (label "ROW2" (at 113.7882 104.013 0)
     (effects (font (size 1.27 1.27)) (justify left bottom))
   )
@@
     (effects (font (size 1.27 1.27)) (justify left bottom))
   )
-  (label "ROW6" (at 113.7882 106.553 0)
+  (label "ROW6" (at 113.7882 93.8522 0)
     (effects (font (size 1.27 1.27)) (justify left bottom))
   )
-  (label "ROW5" (at 113.7882 104.013 0)
+  (label "ROW5" (at 113.7882 96.393 0)
     (effects (font (size 1.27 1.27)) (justify left bottom))
   )
@@
     (effects (font (size 1.27 1.27)) (justify left bottom))
   )
-  (label "ROW3" (at 113.7663 98.933 0)
+  (label "ROW3" (at 113.7663 101.4742 0)
     (effects (font (size 1.27 1.27)) (justify left bottom))
   )
-  (label "COL3" (at 113.8448 91.313 0)
+  (label "COL3" (at 113.7663 109.093 0)
     (effects (font (size 1.27 1.27)) (justify left bottom))
   )
@@
     (effects (font (size 1.27 1.27)) (justify left bottom))
   )
-  (label "ROW7" (at 113.7663 109.093 0)
+  (label "ROW7" (at 113.8448 91.313 0)
     (effects (font (size 1.27 1.27)) (justify left bottom))
   )
-  (label "ROW4" (at 113.7663 101.4742 0)
+  (label "ROW4" (at 113.7663 98.933 0)
     (effects (font (size 1.27 1.27)) (justify left bottom))
   )
@@
     (effects (font (size 1.27 1.27)) (justify left bottom))
   )
-  (label "ROW1" (at 113.7882 93.8522 0)
+  (label "ROW1" (at 113.7882 106.553 0)
     (effects (font (size 1.27 1.27)) (justify left bottom))
   )
