File: pcb/rpad/toroufc-rpad.kicad_sch (KiCad schematic)
At the start: 11 parts, among them J10 Conn_01x06_Male, SW1 SW_Push, SW2 SW_Push, SW3 SW_Push, SW4 SW_Push, SW5 SW_Push

Commit message: Update toroufc-rpad.kicad_sch
Other:
- title: (none) -> TORO UFC v1.0 - Right PAD
Changed lines of the file:
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@@
 (kicad_sch (version 20211123) (generator eeschema)
   (paper "A4")
+  (title_block
+    (title "TORO UFC v1.0 - Right PAD")
+    (date "2022-02-12")
+    (rev "1.0")
+  )
   (junction (at 150.4284 83.185) (diameter 0) (color 0 0 0 0)
   )

Commit message: Preparing PCBs v2
Connections:
- net COL5: now also J10.6 (Pin_6); no longer J10.1 (Pin_1)
- net ROW1: now also J10.5 (Pin_5); no longer J10.2 (Pin_2)
- net ROW2: now also J10.4 (Pin_4); no longer J10.3 (Pin_3)
- net ROW3: now also J10.3 (Pin_3); no longer J10.4 (Pin_4)
- net ROW4: now also J10.2 (Pin_2); no longer J10.5 (Pin_5)
- net ROW5: now also J10.1 (Pin_1); no longer J10.6 (Pin_6)
Changed lines of the file:
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@@
     (stroke (width 0) (type default) (color 0 0 0 0))
   )
-  (label "ROW5" (at 112.2423 91.4412 0)
+  (label "ROW5" (at 112.3208 78.74 0)
     (effects (font (size 1.27 1.27)) (justify left bottom))
   )
@@
     (effects (font (size 1.27 1.27)) (justify left bottom))
   )
-  (label "ROW3" (at 112.2642 86.36 0)
+  (label "ROW3" (at 112.2642 83.8192 0)
     (effects (font (size 1.27 1.27)) (justify left bottom))
   )
-  (label "ROW1" (at 112.3208 81.28 0)
+  (label "ROW1" (at 112.2423 88.9 0)
     (effects (font (size 1.27 1.27)) (justify left bottom))
   )
-  (label "ROW4" (at 112.2423 88.9 0)
+  (label "ROW4" (at 112.3208 81.28 0)
     (effects (font (size 1.27 1.27)) (justify left bottom))
   )
@@
     (effects (font (size 1.27 1.27)) (justify left bottom))
   )
-  (label "ROW2" (at 112.2642 83.8192 0)
+  (label "ROW2" (at 112.2642 86.36 0)
     (effects (font (size 1.27 1.27)) (justify left bottom))
   )
@@
     (effects (font (size 1.27 1.27)) (justify left bottom))
   )
-  (label "COL5" (at 112.3208 78.74 0)
+  (label "COL5" (at 112.2423 91.44 0)
     (effects (font (size 1.27 1.27)) (justify left bottom))
   )
